Commit message: change compensation in ur5.urdf.xacro

File: ur_description/urdf/ur5.urdf.xacro (robot description, xacro)
@@ -285,8 +285,9 @@
       </collision>
     </link>
+<!-- x point to down, y point to me, z point to door -->
     <joint name="${prefix}grasping_fixed_joint" type="fixed">
       <parent link="${prefix}ee_link" />
       <child link = "${prefix}grasping_frame" />
-      <origin xyz="0.25 -0.0353553391 -0.0353553391" rpy="${pi/4.0} 0.0 0.0" />
+      <origin xyz="0.25 0.0 0.0" rpy="${pi/4.0} 0.0 0.0" />
     </joint>
     <link name="${prefix}grasping_frame">

Commit message: add optoforce sensor_link in ur5.urdf.xacro

File: ur_description/urdf/ur5.urdf.xacro (robot description, xacro)
@@ -299,4 +299,17 @@
       </collision>
     </link>
+    <joint name="${prefix}sensor_joint" type="fixed">
+      <parent link="${prefix}tool0" />
+      <child link = "${prefix}sensor_link" />
+      <origin xyz="0.0 0.0 0.035" rpy="0.0 0.0 0.0" />
+    </joint>
+    <link name="${prefix}sensor_link">
+      <collision>
+        <geometry>
+          <box size="0.01 0.01 0.01"/>
+        </geometry>
+        <origin rpy="0 0 0" xyz="0.0 0 0"/>
+      </collision>
+    </link>
     <xacro:ur_arm_transmission prefix="${prefix}" />
     <xacro:ur_arm_gazebo prefix="${prefix}" />
